File: schematic/amplifeuer-schematic-psu.sch (KiCad schematic (older format))
At the start: 10 parts, among them J6 Power out, J7 Power in, U2 LT1071

Commit message: Concretise PSU schematic, with thanks to NimbleJack3. Add status LEDs to PSU. Add second filter stage to PSU
Parts:
- added C14: 100μF, Capacitor_THT:CP_Radial_D8.0mm_P2.50mm, symbol Device:CP
- added C15: 100nF, Capacitor_THT:C_Disc_D7.5mm_W2.5mm_P5.00mm, symbol Device:C
- added D12: Red, LED_THT:LED_Rectangular_W5.0mm_H2.0mm, symbol Device:LED
- added D13: Green, LED_THT:LED_Rectangular_W5.0mm_H2.0mm, symbol Device:LED
- added L12: 10μH, Battery:BatteryHolder_Keystone_2479_3xAAA, symbol Device:L_Core_Ferrite
- added R12: 2200R, Resistor_THT:R_Axial_DIN0204_L3.6mm_D1.6mm_P5.08mm_Horizontal, symbol Device:R
- C11: renamed from C10; footprint Capacitor_THT:CP_Radial_D6.3mm_P2.50mm -> Capacitor_THT:CP_Radial_D8.0mm_P2.50mm
- C12: renamed from C11; footprint Capacitor_THT:CP_Radial_D5.0mm_P2.50mm -> Battery:BatteryHolder_Keystone_2479_3xAAA
- D11: renamed from D1; value D_Schottky -> 1N5822; footprint Diode_THT:D_5KPW_P7.62mm_Vertical_AnodeUp -> Battery:BatteryHolder_Keystone_2479_3xAAA
- L11: renamed from L1; value L_Core_Ferrite -> 100..200μH?; footprint Inductor_THT:L_Axial_L16.0mm_D9.5mm_P5.08mm_Vertical_Vishay_IM-10-37 -> Battery:BatteryHolder_Keystone_2479_3xAAA
- RV11: renamed from RV1; value R_POT_TRIM -> 5000RTRIM
- renumbered C12 to C13, J6 to J11, J7 to J12, R3 to R11, U2 to U11
Connections:
- wire segments 10 -> 13
Other:
- note removed: "TODO: P/N / value?"
- note removed: "TODO: Vc network?"
- note removed: "TODO: which diode?"

Commit message: Stabilise components and their footprints
Parts:
- C12: footprint Battery:BatteryHolder_Keystone_2479_3xAAA -> Capacitor_THT:C_Disc_D4.7mm_W2.5mm_P5.00mm
- C13: Variant (none) -> Low ESR
- D11: footprint Battery:BatteryHolder_Keystone_2479_3xAAA -> Diode_THT:D_DO-201AD_P5.08mm_Vertical_AnodeUp
- L11: value 100..200μH? -> 100μH; footprint Battery:BatteryHolder_Keystone_2479_3xAAA -> Inductor_THT:L_Toroid_Vertical_L14.5mm_W7.0mm_P7.18mm; I_max (none) -> 3A
- L12: footprint Battery:BatteryHolder_Keystone_2479_3xAAA -> Inductor_THT:L_Radial_D6.8mm_5.0mm_P2.54mm_sleeved
Changed lines of the file:
@@
 U 1 1 5D49B3ED
 P 6400 3350
-F 0 "C13" H 6518 3396 50  0000 L CNN
-F 1 "1000μF" H 6518 3305 50  0000 L CNN
+F 0 "C13" H 6518 3441 50  0000 L CNN
+F 1 "1000μF" H 6518 3350 50  0000 L CNN
 F 2 "Capacitor_THT:CP_Radial_D10.0mm_P5.00mm" H 6438 3200 50  0001 C CNN
 F 3 "~" H 6400 3350 50  0001 C CNN
+F 4 "Low ESR" H 6518 3259 50  0000 L CNN "Variant"
 	1    6400 3350
 	1    0    0    -1
@@
 F 0 "D11" H 6150 2984 50  0000 C CNN
 F 1 "1N5822" H 6150 3075 50  0000 C CNN
-F 2 "Battery:BatteryHolder_Keystone_2479_3xAAA" H 6150 3200 50  0001 C CNN
+F 2 "Diode_THT:D_DO-201AD_P5.08mm_Vertical_AnodeUp" H 6150 3200 50  0001 C CNN
 F 3 "~" H 6150 3200 50  0001 C CNN
 	1    6150 3200
@@
 U 1 1 5D49BC9C
 P 5700 3000
-F 0 "L11" V 5925 3000 50  0000 C CNN
-F 1 "100..200μH?" V 5834 3000 50  0000 C CNN
-F 2 "Battery:BatteryHolder_Keystone_2479_3xAAA" H 5700 3000 50  0001 C CNN
+F 0 "L11" V 6016 3000 50  0000 C CNN
+F 1 "100μH" V 5925 3000 50  0000 C CNN
+F 2 "Inductor_THT:L_Toroid_Vertical_L14.5mm_W7.0mm_P7.18mm" H 5700 3000 50  0001 C CNN
 F 3 "~" H 5700 3000 50  0001 C CNN
+F 4 "3A" V 5834 3000 50  0000 C CNN "I_max"
 	1    5700 3000
 	0    -1   -1   0
@@
 F 0 "C12" H 5665 4346 50  0000 L CNN
 F 1 "1μF" H 5665 4255 50  0000 L CNN
-F 2 "Battery:BatteryHolder_Keystone_2479_3xAAA" H 5588 4150 50  0001 C CNN
+F 2 "Capacitor_THT:C_Disc_D4.7mm_W2.5mm_P5.00mm" H 5588 4150 50  0001 C CNN
 F 3 "~" H 5550 4300 50  0001 C CNN
 	1    5550 4300
@@
 F 0 "L12" V 6875 3200 50  0000 C CNN
 F 1 "10μH" V 6784 3200 50  0000 C CNN
-F 2 "Battery:BatteryHolder_Keystone_2479_3xAAA" H 6650 3200 50  0001 C CNN
+F 2 "Inductor_THT:L_Radial_D6.8mm_5.0mm_P2.54mm_sleeved" H 6650 3200 50  0001 C CNN
 F 3 "~" H 6650 3200 50  0001 C CNN
 	1    6650 3200

Commit message: Add heatsink to PSU schematic
Parts:
- added HS11: Aavid-5342B, Heatsink:Heatsink_Aavid-5342-TO220_Vertical, symbol Mechanical:Heatsink_Pad
Changed lines of the file:
@@
+	1    0    0    -1
+$EndComp
+$Comp
+L Mechanical:Heatsink_Pad HS11
+U 1 1 5D4D71C9
+P 5500 2400
+F 0 "HS11" H 5641 2441 50  0000 L CNN
+F 1 "Aavid-5342B" H 5641 2350 50  0000 L CNN
+F 2 "Heatsink:Heatsink_Aavid-5342-TO220_Vertical" H 5512 2350 50  0001 C CNN
+F 3 "~" H 5512 2350 50  0001 C CNN
+	1    5500 2400
+	1    0    0    -1
+$EndComp
+$Comp
+L power:GND #PWR0103
+U 1 1 5D4D73F1
+P 5500 2500
+F 0 "#PWR0103" H 5500 2250 50  0001 C CNN
+F 1 "GND" H 5505 2327 50  0000 C CNN
+F 2 "" H 5500 2500 50  0001 C CNN
+F 3 "" H 5500 2500 50  0001 C CNN
+	1    5500 2500
 	1    0    0    -1
 $EndComp
