File: schematic/amplifeuer-schematic-psu.sch (KiCad schematic (older format))
At the start: 17 parts, among them J11 Power out, J12 Power in, U11 LT1071

Commit message: Lay out PSU
Parts:
- R12: footprint Resistor_THT:R_Axial_DIN0204_L3.6mm_D1.6mm_P5.08mm_Horizontal -> Resistor_THT:R_Axial_DIN0204_L3.6mm_D1.6mm_P7.62mm_Horizontal
Changed lines of the file:
@@
 F 0 "R12" H 4170 3646 50  0000 L CNN
 F 1 "2200R" H 4170 3555 50  0000 L CNN
-F 2 "Resistor_THT:R_Axial_DIN0204_L3.6mm_D1.6mm_P5.08mm_Horizontal" V 4030 3600 50  0001 C CNN
+F 2 "Resistor_THT:R_Axial_DIN0204_L3.6mm_D1.6mm_P7.62mm_Horizontal" V 4030 3600 50  0001 C CNN
 F 3 "~" H 4100 3600 50  0001 C CNN
 	1    4100 3600
